File: ControlA/MECANIQUE.kicad_sch (KiCad schematic)
At the start: 0 parts

Commit message: final shema symbole
Parts:
- added H1, H2, H3, H4: MountingHole_Pad, MountingHole:MountingHole_4.3mm_M4_Pad_Via, symbol Mechanical:MountingHole_Pad
- added R69, R70, R71, R72: 0R, Resistor_SMD:R_0805_2012Metric, symbol Device:R
Connections:
- new net: H4.1, R72.1
- new net: H2.1, R70.1
- new net: H3.1, R71.1
- new net: H1.1, R69.1
- new net GND: R69.2, R70.2, R71.2, R72.2
Other:
- note added: "FIT A ZERO OMH LINK , CAP ,OR RESISTOR"
- note added: "MECANIQUE"
- note added: "MOUNTING HOLES"
