File: ControlA/Step_Dowun_Convert.kicad_sch (KiCad schematic)
At the start: 0 parts

Commit message: final shema symbole
Parts:
- added C5, C6, C7, C8: 1u, Capacitor_SMD:C_0805_2012Metric, symbol Device:C
- added D3, D5: LED, footprint:LED0805-R-RD, symbol Device:LED
- added D4: BAT60A, Diode_SMD:D_SOD-323, symbol Diode:BAT60A
- added R5: 1K, Resistor_SMD:R_0805_2012Metric, symbol Device:R
- added R6: 1k, Resistor_SMD:R_0805_2012Metric, symbol Device:R
- added U2: AMS1117-3.3, Package_TO_SOT_SMD:SOT-223-3_TabPin2, symbol Regulator_Linear:AMS1117-3.3
Connections:
- new net: D3.2 (A), R5.2
- new net: D5.2 (A), R6.2
- new net +3V3: D4.1 (K), R6.1
- new net +3V3_IC: C7.1, C8.1, D4.2 (A), U2.2 (VO)
- new net +5V: C5.1, C6.1, R5.1, U2.3 (VI)
- new net GND: C5.2, C6.2, C7.2, C8.2, D3.1 (K), D5.1 (K), U2.1 (GND)
Other:
- note added: "FROM MOSFET DRIVER OR EXTERNAL"
- note added: "STEP DOWN CONVERT"

Commit message: CHANGE V11
change v1
Parts:
- C5, C6, C7, C8: footprint Capacitor_SMD:C_0805_2012Metric -> Capacitor_SMD:C_0603_1608Metric
Changed lines of the file:
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@@
 			)
 		)
-		(property "Footprint" "Capacitor_SMD:C_0805_2012Metric"
+		(property "Footprint" "Capacitor_SMD:C_0603_1608Metric"
 			(at 105.1052 81.28 0)
 			(effects
@@
 			)
 		)
-		(property "Footprint" "Capacitor_SMD:C_0805_2012Metric"
+		(property "Footprint" "Capacitor_SMD:C_0603_1608Metric"
 			(at 152.0952 81.28 0)
 			(effects
@@
 			)
 		)
-		(property "Footprint" "Capacitor_SMD:C_0805_2012Metric"
+		(property "Footprint" "Capacitor_SMD:C_0603_1608Metric"
 			(at 138.1252 81.28 0)
 			(effects
@@
 			)
 		)
-		(property "Footprint" "Capacitor_SMD:C_0805_2012Metric"
+		(property "Footprint" "Capacitor_SMD:C_0603_1608Metric"
 			(at 91.1352 81.28 0)
 			(effects
