File: ControlA/MOSFTs.kicad_sch (KiCad schematic)
At the start: 0 parts

Commit message: final shema symbole
Parts:
- added C61, C62: 2n2, Capacitor_SMD:C_0805_2012Metric, symbol Device:C
- added Q1, Q2, Q3, Q4, Q5, Q6: HSBA15810C, footprint:PQFN-8_L6.0-W5.0-P1.27-LS6.0-BL, symbol HSBA15810C:HSBA15810C
- added R54, R55, R61, R62: 100R, Resistor_SMD:R_0805_2012Metric, symbol Device:R
- added R56, R57, R60, R63, R66, R67: 4R7, Resistor_SMD:R_0805_2012Metric, symbol Device:R
- added R58, R64, R68: 39K, Resistor_SMD:R_0805_2012Metric, symbol Device:R
- added R59, R65: 0R001, Resistor_SMD:R_0805_2012Metric, symbol Device:R
Connections:
- new net +VDC: Q1.3 (S), Q3.3 (S), Q5.3 (S)
- new net GND: Q6.5 (D), R55.2, R58.1, R59.1, R62.2, R64.1, R65.1, R68.1
- new net H1_LOW: Q2.6 (D), R54.2, R59.2
- new net H1_VS: Q1.9 (D), Q2.3 (S)
- new net H2_LOW: Q4.6 (D), R61.2, R65.2
- new net H2_VS: Q3.9 (D), Q4.3 (S)
- new net H3_VS: Q5.9 (D), Q6.3 (S)
- new net M_H1: R56.1
- new net M_H1_RG: Q1.4 (G), R56.2
- new net M_H2: R60.1
- new net M_H2_RG: Q3.4 (G), R60.2
- new net M_H3: R66.1
- new net M_H3_RG: Q5.4 (G), R66.2
- new net M_L1: R57.1
- new net M_L1_RG: Q2.4 (G), R57.2, R58.2
- new net M_L2: R63.1
- new net M_L2_RG: Q4.4 (G), R63.2, R64.2
- new net M_L3: R67.1
- new net M_L3_RG: Q6.4 (G), R67.2, R68.2
- new net S1_N: C61.1, R54.1
- new net S1_P: C61.2, R55.1
- new net S2_N: C62.1, R61.1
- new net S2_P: C62.2, R62.1
- no-connect marks 0 -> 36
Other:
- note added: "MOSFET"
- note added: "PLACE AS CLOSE AS POSSIBLE TO THE BULK CAPACITANCE"
- note added: "Q_SOURCES"
- note added: "ROUTE AS KELVING CONNECTIONS"

Commit message: CHANGE V11
change v1
Parts:
- C61, C62: footprint Capacitor_SMD:C_0805_2012Metric -> Capacitor_SMD:C_0603_1608Metric
Changed lines of the file:
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@@
 			)
 		)
-		(property "Footprint" "Capacitor_SMD:C_0805_2012Metric"
+		(property "Footprint" "Capacitor_SMD:C_0603_1608Metric"
 			(at 78.4352 129.54 0)
 			(effects
@@
 			)
 		)
-		(property "Footprint" "Capacitor_SMD:C_0805_2012Metric"
+		(property "Footprint" "Capacitor_SMD:C_0603_1608Metric"
 			(at 152.0952 129.54 0)
 			(effects

Commit message: connector
add conctor power mosft
Parts:
- added J5, J6, J7: Conn_01x01, footprint:7461097, symbol Connector_Generic:Conn_01x01
Connections:
- net M_H2_RG is gone; now on net +VDC: Q3.4 (G), R60.2
- net H1_VS: now also J5.1 (Pin_1)
- net H2_VS: now also J6.1 (Pin_1)
- net H3_VS: now also J7.1 (Pin_1)
Other:
- note added: "output phase1"
- note added: "output phase2"
- note added: "output phase3"
- moved on the sheet: C61, C62, Q1, Q2, Q3, Q4, Q5, Q6, R54, R55, R56, R57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
