File: ControlA/ControlA.kicad_pcb (KiCad board)
At the start: 4 copper layers, 111.6 x 78.8 mm, 167 parts, among them CN1 PH-4A_RHOS, J1 XT30PW-M, J2 Conn_01x08, J3 Conn_01x06, J4 Conn_01x03, J5 Conn_01x01, J6 Conn_01x01, J7 Conn_01x01, Q1 HSBA15810C, Q2 HSBA15810C, Q3 HSBA15810C, Q4 HSBA15810C, Q5 HSBA15810C, Q6 HSBA15810C, SW1 TS-KG87S-AT15F, U1 XH-2PWBPZ, U10 YSPI0530-220M, U2 AMS1117-3.3, U3 STM32F405RGTx, U4 DRV8302DCAR, U5 ESDCAN24-2BLY, U6 744227S, U7 SN65HVD230D, U8 B06B-PARK-1_(LF)(SN), U9 TYPE-C_16PIN_2MD(073), Y1 Crystal

Commit message: change layour boedrer
change layout broder
Parts:
- moved R40 118.3 mm to (155.0, 120.9)
- moved D1 105.6 mm to (128.9, 110.0)
- moved C54 103.8 mm to (138.0, 109.9)
- moved C5 93.8 mm to (151.2, 106.5)
- moved C6 93.8 mm to (154.2, 106.5)
- moved C7 93.8 mm to (160.2, 115.0)
- moved C8 93.8 mm to (160.2, 117.5)
- moved D3 93.8 mm to (148.2, 112.1)
- moved D5 93.8 mm to (165.7, 116.6)
- moved R5 93.8 mm to (148.7, 106.4)
- moved U2 93.8 mm to (160.7, 109.2)
- moved H2 19.7 mm to (167.3, 53.0)
Other:
- board size 111.6 x 78.8 mm -> 131.9 x 81.5 mm
Changed lines of the file:
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@@
 	(footprint "footprint:LED0805-R-RD"
 		(layer "F.Cu")
-		(at 85.8 42.050294 -90)
+		(at 148.2 112.050294 -90)
 		(descr "LED0805-R-RD footprint")
 		(tags "LED0805-R-RD footprint C98221")
@@
 	(footprint "Resistor_SMD:R_0805_2012Metric"
 		(layer "F.Cu")
-		(at 86.3 36.412501 -90)
+		(at 148.7 106.412501 -90)
 		(descr "Resistor SMD 0805 (2012 Metric), square (rectangular) end terminal, IPC_7351 nominal, (Body size source: IPC-SM-782 page 72, https://www.pcb-3d.com/wordpress/wp-content/uploads/ipc-sm-782a_amendment_1_and_2.pdf), generated with kicad-footprint-generator")
 		(tags "resistor")
@@
 	(footprint "Capacitor_SMD:C_0603_1608Metric"
 		(layer "F.Cu")
-		(at 43.8 66.23)
+		(at 137.99 109.91)
 		(descr "Capacitor SMD 0603 (1608 Metric), square (rectangular) end terminal, IPC_7351 nominal, (Body size source: IPC-SM-782 page 76, https://www.pcb-3d.com/wordpress/wp-content/uploads/ipc-sm-782a_amendment_1_and_2.pdf), generated with kicad-footprint-generator")
 		(tags "capacitor")
@@
 	(footprint "Capacitor_SMD:C_0603_1608Metric"
 		(layer "F.Cu")
-		(at 88.8 36.45 -90)
+		(at 151.2 106.45 -90)
 		(descr "Capacitor SMD 0603 (1608 Metric), square (rectangular) end terminal, IPC_7351 nominal, (Body size source: IPC-SM-782 page 76, https://www.pcb-3d.com/wordpress/wp-content/uploads/ipc-sm-782a_amendment_1_and_2.pdf), generated with kicad-footprint-generator")
 		(tags "capacitor")
@@
 	(footprint "Package_TO_SOT_SMD:SOT-223-3_TabPin2"
 		(layer "F.Cu")
-		(at 98.3 39.15 -90)
+		(at 160.7 109.15 -90)
 		(descr "module CMS SOT223 4 pins")
 		(tags "CMS SOT")
@@
 	(footprint "footprint:LED0805-R-RD"
 		(layer "F.Cu")
-		(at 103.3 46.550294 90)
+		(at 165.7 116.550294 90)
 		(descr "LED0805-R-RD footprint")
 		(tags "LED0805-R-RD footprint C98221")
@@
 	(footprint "MountingHole:MountingHole_4.3mm_M4_Pad_Via"
 		(layer "F.Cu")
-		(at 185.18 61.25)
+		(at 167.260419 52.950419)
 		(descr "Mounting Hole 4.3mm, M4")
 		(tags "mounting hole 4.3mm m4")
@@
 	(footprint "Resistor_SMD:R_0805_2012Metric"
 		(layer "F.Cu")
-		(at 49.9 66.667501 90)
+		(at 155 120.9125 90)
 		(descr "Resistor SMD 0805 (2012 Metric), square (rectangular) end terminal, IPC_7351 nominal, (Body size source: IPC-SM-782 page 72, https://www.pcb-3d.com/wordpress/wp-content/uploads/ipc-sm-782a_amendment_1_and_2.pdf), generated with kicad-footprint-generator")
 		(tags "resistor")
@@
 	(footprint "Capacitor_SMD:C_0603_1608Metric"
 		(layer "F.Cu")
-		(at 91.8 36.45 -90)
+		(at 154.2 106.45 -90)
 		(descr "Capacitor SMD 0603 (1608 Metric), square (rectangular) end terminal, IPC_7351 nominal, (Body size source: IPC-SM-782 page 76, https://www.pcb-3d.com/wordpress/wp-content/uploads/ipc-sm-782a_amendment_1_and_2.pdf), generated with kicad-footprint-generator")
 		(tags "capacitor")
@@
 	(footprint "Capacitor_SMD:C_0603_1608Metric"
 		(layer "F.Cu")
-		(at 97.85 47.500001)
+		(at 160.25 117.500001)
 		(descr "Capacitor SMD 0603 (1608 Metric), square (rectangular) end terminal, IPC_7351 nominal, (Body size source: IPC-SM-782 page 76, https://www.pcb-3d.com/wordpress/wp-content/uploads/ipc-sm-782a_amendment_1_and_2.pdf), generated with kicad-footprint-generator")
 		(tags "capacitor")
@@
 	(footprint "Capacitor_SMD:C_0603_1608Metric"
 		(layer "F.Cu")
-		(at 97.85 45.000001)
+		(at 160.25 115.000001)
 		(descr "Capacitor SMD 0603 (1608 Metric), square (rectangular) end terminal, IPC_7351 nominal, (Body size source: IPC-SM-782 page 76, https://www.pcb-3d.com/wordpress/wp-content/uploads/ipc-sm-782a_amendment_1_and_2.pdf), generated with kicad-footprint-generator")
 		(tags "capacitor")
@@
 	(footprint "footprint:DIOM4325X250N"
 		(layer "F.Cu")
-		(at 40 53 -90)
+		(at 128.94 110.02 -90)
 		(property "Reference" "D1"
 			(at -0.925 -2.43 90)
@@
 		)
 	)
-	(gr_line
-		(start 161.58 51.181068)
-		(end 161.58 129.98)
-		(stroke
-			(width 0.05)
-			(type default)
-		)
-		(layer "Edge.Cuts")
-	)
 	(gr_rect
-		(start 71 61)
-		(end 114 104)
+		(start 48.59 47.67)
+		(end 180.5 129.21)
 		(stroke
 			(width 0.05)
@@
 		(layer "Edge.Cuts")
 	)
-	(gr_line
-		(start 161.58 51.181068)
-		(end 59.951068 51.181068)
-		(stroke
-			(width 0.05)
-			(type default)
-		)
-		(layer "Edge.Cuts")
-	)
-	(gr_line
-		(start 60 130)
-		(end 161.59 130)
-		(stroke
-			(width 0.05)
-			(type default)
-		)
-		(layer "Edge.Cuts")
-	)
-	(gr_arc
-		(start 49.951068 61.181068)
-		(mid 52.88 54.11)
-		(end 59.951068 51.181068)
-		(stroke
-			(width 0.05)
-			(type default)
-		)
-		(layer "Edge.Cuts")
-	)
-	(gr_arc
-		(start 60 130)
-		(mid 52.928932 127.071068)
-		(end 50 120)
-		(stroke
-			(width 0.05)
-			(type default)
-		)
-		(layer "Edge.Cuts")
-	)
-	(gr_line
-		(start 49.951068 61.181068)
-		(end 49.951068 120)
-		(stroke
-			(width 0.05)
-			(type default)
-		)
-		(layer "Edge.Cuts")
-	)
